Commit message: Update A1 for noetic/focal
Update husky urdf and rviz config

Update rviz config

File: wall_following_assignment/urdf/accessories/sick_lms1xx_mount.urdf.xacro (robot description, xacro)
@@ -28,5 +28,5 @@
   <xacro:include filename="$(find lms1xx)/urdf/sick_lms1xx.urdf.xacro" />
   <xacro:macro name="sick_lms1xx_mount" params="prefix topic">
-  <sick_lms1xx frame="${prefix}_laser" topic="${topic}" />
+  <xacro:sick_lms1xx frame="${prefix}_laser" topic="${topic}" />
     <link name="${prefix}_laser_mount">
       <visual>

File: wall_following_assignment/urdf/husky.urdf.xacro (robot description, xacro)
@@ -30,9 +30,9 @@
   <!--xacro:include filename="$(find ur_description)/urdf/ur5.urdf.xacro" /-->
   <!--xacro:include filename="$(find velodyne_description)/urdf/VLP-16.urdf.xacro" /-->
-  <property name="M_PI" value="3.14159"/>
+  <xacro:property name="M_PI" value="3.14159"/>
   <!-- Base Size -->
-  <property name="base_x_size" value="0.98740000" />
-  <property name="base_y_size" value="0.57090000" />
-  <property name="base_z_size" value="0.24750000" />
+  <xacro:property name="base_x_size" value="0.98740000" />
+  <xacro:property name="base_y_size" value="0.57090000" />
+  <xacro:property name="base_z_size" value="0.24750000" />
   <!-- Wheel Mounting Positions -->
   <xacro:property name="wheelbase" value="0.5120" />
@@ -120,5 +120,5 @@
     </xacro:if>
     <xacro:if value="$(arg laser_enabled)">
-      <sick_lms1xx_mount prefix="base" topic="scan"/>
+      <xacro:sick_lms1xx_mount prefix="base" topic="scan"/>
       <joint name="laser_mount_joint" type="fixed">
         <origin xyz="$(optenv HUSKY_LMS1XX_XYZ 0.2206 0.0 0.00635)"
